File: rtc/kicad/rtc.kicad_sch (KiCad schematic)
At the start: 10 parts, among them J1 Conn_RIOT, Q1 2N3904, U1 DS1305N, Y1 32.768khz

Commit message: Change transistor pads to make soldering easier
Parts:
- Q1: footprint Package_TO_SOT_THT:TO-92_Inline -> Package_TO_SOT_THT:TO-92_Inline_Wide
Changed lines of the file:
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@@
     (title "PAL-1 Real Time Clock")
     (date "Feb 2024")
-    (rev "1.0a")
+    (rev "${VERSION}")
     (company "Plastic Objects Limited")
   )
@@
       (effects (font (size 1.27 1.27)) (justify left))
     )
-    (property "Footprint" "Package_TO_SOT_THT:TO-92_Inline" (at 116.84 120.015 0)
+    (property "Footprint" "Package_TO_SOT_THT:TO-92_Inline_Wide" (at 116.84 120.015 0)
       (effects (font (size 1.27 1.27) italic) (justify left) hide)
     )
