File: speech/kicad/speech.kicad_pcb (KiCad board)
At the start: 2 copper layers, 57 x 39 mm, 22 parts, among them J1 Conn_RIOT, J2 AudioJack3_Ground, Q1 BC557, U1 SP0256AL2, U2 LM386, Y1 3.12Mhz

Commit message: Update schematic and board layout
Parts:
- removed D1: 1N914, Diode_THT:D_DO-35_SOD27_P7.62mm_Horizontal
- removed Q1: BC557, Package_TO_SOT_THT:TO-92_Inline_Wide
- removed the R4 at (135.1, 87.9)
- added C2: 0.1uF, Capacitor_THT:C_Disc_D3.0mm_W1.6mm_P2.50mm, F.Cu at (142.2, 102.6)
- moved R1 5.59 mm to (142.2, 99.8)
- moved J2 1.27 mm to (114.5, 91.2)
- moved RV1 1.03 mm to (129.8, 98.7)
- renumbered C2 to C3, C3 to C4, C4 to C5, C5 to C6, C6 to C7, C7 to C8, C8 to C9, R5 to R4
Connections:
- net SBY renamed ~{BUSY}
- net ~{LRQ} renamed ~{LOAD}
- C1 pad 1: Net-(D1-A) -> ~{RESET}
- C7 pad 1: Net-(Q1-C) -> VCC
- J1 pad 15: PB6 -> ~{STROBE}
- J1 pad 17: PB7 -> ~{RESET}
- J1 pad 4: PA0 -> unconnected-(J1-Pin_4-Pad4)
- R1 pad 2: Net-(D1-A) -> ~{RESET}
- U1 pad 10: PB7 -> GND
- U1 pad 11: PB6 -> GND
- U1 pad 2: Net-(D1-A) -> ~{RESET}
- U1 pad 20: PA0 -> ~{STROBE}
- U1 pad 25: Net-(D1-A) -> ~{RESET}
- U2 pad 6: Net-(Q1-C) -> VCC
Routing:
- net ~{RESET}: track 0.00 -> 93.4 mm
- net Net-(D1-A): track 89.4 -> 0.00 mm
- net PB6: track 59.0 -> 0.00 mm
- net PB7: track 55.6 -> 0.00 mm
- net ~{STROBE}: track 0.00 -> 46.0 mm
- net PA0: track 41.9 -> 0.00 mm
- net Net-(Q1-C): track 23.6 -> 0.00 mm
- net Net-(Q1-B): track 10.5 -> 0.00 mm
- net Net-(U2-+): track 19.5 -> 9.52 mm
- net VCC: track 86.5 -> 81.4 mm
- net ~{BUSY}: track 74.7 -> 71.2 mm
- net ~{LOAD}: track 74.3 -> 72.2 mm
- net PB3: track 48.1 -> 46.7 mm
- net PB2: track 47.9 -> 46.5 mm
- net PB1: track 47.7 -> 46.4 mm
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- removed copper zone on B.Cu, net (none)
Other:
- board text added: "v1.0A"
