File: speech/kicad/speech.kicad_sch (KiCad schematic)
At the start: 21 parts, among them J1 Conn_RIOT, J2 AudioJack3_Ground, Q1 BC557, U1 SP0256AL2, U2 LM386, Y1 3.12Mhz

Commit message: Update schematic and board layout
Parts:
- removed D1: 1N914, Diode_THT:D_DO-35_SOD27_P7.62mm_Horizontal, symbol Diode:1N914
- removed Q1: BC557, Package_TO_SOT_THT:TO-92_Inline_Wide, symbol Simulation_SPICE:PNP
- removed R4: 1K, Resistor_THT:R_Axial_DIN0207_L6.3mm_D2.5mm_P7.62mm_Horizontal, symbol Device:R
- added C2: 0.1uF, Capacitor_THT:C_Disc_D3.0mm_W1.6mm_P2.50mm, symbol Device:C_Small
- renumbered C2 to C3, C3 to C4, C4 to C5, C5 to C6, C6 to C7, C7 to C8, C8 to C9, R5 to R4
Connections:
- net GND: now also U1.10 (A8), U1.11 (A7), C2.2
- net VCC: now also C7.1, U2.6 (V+), C2.1
- net ~{RESET}: now reaches C1.1, R1.2, U1.2 (~{RESET}), U1.25 (~{SBY_RST})
- net ~{RESET}: now also J1.17 (Pin_17)
- net PA0: no longer names the net of J1.4 (Pin_4)
- net PA0: no longer U1.20 (~{ALD})
- net PB6 renamed ~{STROBE}
- net ~{STROBE}: now also U1.20 (~{ALD}); no longer U1.11 (A7)
- removed net PB7: J1.17 (Pin_17), U1.10 (A8)
- net SBY renamed ~{BUSY}
- net ~{LRQ} renamed ~{LOAD}
- no-connect marks 16 -> 17
Other:
- moved on the sheet: C1
